Commit message: [feat][ros2][sim]: Implement fully  4 legs gait

File: Software/Middleware/robot_ros2/src/simulation/urdf/test.urdf (robot description, URDF)
Before this commit: robot 3dof_leg, 4 links, 3 joints
Links:
- removed link link1
- removed link link2
- removed link link3
- added link body_link; visual box size=0.3 0.18049 0.06
- added link link_lb_1; visual box size=0.01 0.046 0.01
- added link link_lb_2; visual box size=0.1063 0.01 0.01
- added link link_lb_3; visual box size=0.10403 0.01 0.01
- added link link_lf_1; visual box size=0.01 0.046 0.01
- added link link_lf_2; visual box size=0.1063 0.01 0.01
- added link link_lf_3; visual box size=0.10403 0.01 0.01
- added link link_rb_1; visual box size=0.01 0.046 0.01
- added link link_rb_2; visual box size=0.1063 0.01 0.01
- added link link_rb_3; visual box size=0.10403 0.01 0.01
- added link link_rf_1; visual box size=0.01 0.046 0.01
- added link link_rf_2; visual box size=0.1063 0.01 0.01
- added link link_rf_3; visual box size=0.10403 0.01 0.01
Joints:
- removed joint joint1
- removed joint joint2
- removed joint joint3
- added joint body_joint: type fixed, parent world_link, child body_link, origin xyz=0 0 0.5
- added joint joint_lb_1: type revolute, parent body_link, child link_lb_1, origin xyz=-0.11014   0.07169   0.00026 rpy= 0        -1.57     -3.14   , axis  0         0         1      , limit lower=-1.57 upper= 1.57 effort=   10 velocity=    1
- added joint joint_lb_2: type revolute, parent link_lb_1, child link_lb_2, origin xyz=0    -0.046    0 rpy=1.57  3.14     0, axis 0     0        1, limit lower=-6.28 upper=6.28 effort=  10 velocity=   1
- added joint joint_lb_3: type revolute, parent link_lb_2, child link_lb_3, origin xyz=-0.1063 0 0 rpy= 0      0 0, axis  0      0 1, limit lower=-6.28 upper=6.28 effort=  10 velocity=   1
- added joint joint_lf_1: type revolute, parent body_link, child link_lf_1, origin xyz=0.11014   0.07169   0.00026 rpy=0        -1.57     -3.14   , axis 0         0         1      , limit lower=-1.57 upper= 1.57 effort=   10 velocity=    1
- added joint joint_lf_2: type revolute, parent link_lf_1, child link_lf_2, origin xyz=0    -0.046    0 rpy=1.57  3.14     0, axis 0     0        1, limit lower=-6.28 upper=6.28 effort=  10 velocity=   1
- added joint joint_lf_3: type revolute, parent link_lf_2, child link_lf_3, origin xyz=-0.1063 0 0 rpy= 0      0 0, axis  0      0 1, limit lower=-6.28 upper=6.28 effort=  10 velocity=   1
- added joint joint_rb_1: type revolute, parent body_link, child link_rb_1, origin xyz=-0.11014  -0.07169   0.00026 rpy= 0        -1.57      0   , axis  0         0         1      , limit lower=-1.57 upper= 1.57 effort=   10 velocity=    1
- added joint joint_rb_2: type revolute, parent link_rb_1, child link_rb_2, origin xyz=0    -0.046   0 rpy=-1.57 0    3.14, axis 0     0       1, limit lower=-6.28 upper=6.28 effort=  10 velocity=   1
- added joint joint_rb_3: type revolute, parent link_rb_2, child link_rb_3, origin xyz=-0.1063 0 0 rpy= 0      0 0, axis  0      0 1, limit lower=-6.28 upper=6.28 effort=  10 velocity=   1
- added joint joint_rf_1: type revolute, parent body_link, child link_rf_1, origin xyz=0.11014  -0.07169   0.00026 rpy=0        -1.57      0   , axis 0         0         1      , limit lower=-1.57 upper= 1.57 effort=   10 velocity=    1
- added joint joint_rf_2: type revolute, parent link_rf_1, child link_rf_2, origin xyz= 0    -0.046 0    rpy=-1.57  0     3.14, axis  0     0     1   , limit lower=-6.28 upper=6.28 effort=  10 velocity=   1
- added joint joint_rf_3: type revolute, parent link_rf_2, child link_rf_3, origin xyz=-0.1063 0 0 rpy= 0      0 0, axis  0      0 1, limit lower=-6.28 upper=6.28 effort=  10 velocity=   1

Commit message: [feat][ros2][sim]: Create the URDF file

File: Software/Middleware/robot_ros2/src/simulation/urdf/test.urdf (robot description, URDF)
Before this commit: robot 3dof_leg, 14 links, 13 joints
Links:
- link body_link: mass None -> 1.0; geometry collision box size=0.3 0.18049 0.06; visual box size=0.3 0.18049 0.06
- link link_lb_1: mass None -> 0.08; geometry collision box size=0.01 0.046 0.01; visual box size=0.01 0.046 0.01
- link link_lb_2: mass None -> 0.09; geometry collision box size=0.1063 0.01 0.01; visual box size=0.1063 0.01 0.01
- link link_lb_3: mass None -> 0.02; geometry collision box size=0.10403 0.01 0.01; visual box size=0.10403 0.01 0.01
- link link_lf_1: mass None -> 0.08; geometry collision box size=0.01 0.046 0.01; visual box size=0.01 0.046 0.01
- link link_lf_2: mass None -> 0.09; geometry collision box size=0.1063 0.01 0.01; visual box size=0.1063 0.01 0.01
- link link_lf_3: mass None -> 0.02; geometry collision box size=0.10403 0.01 0.01; visual box size=0.10403 0.01 0.01
- link link_rb_1: mass None -> 0.08; geometry collision box size=0.01 0.046 0.01; visual box size=0.01 0.046 0.01
- link link_rb_2: mass None -> 0.09; geometry collision box size=0.1063 0.01 0.01; visual box size=0.1063 0.01 0.01
- link link_rb_3: mass None -> 0.02; geometry collision box size=0.10403 0.01 0.01; visual box size=0.10403 0.01 0.01
- link link_rf_1: mass None -> 0.08; geometry collision box size=0.01 0.046 0.01; visual box size=0.01 0.046 0.01
- link link_rf_2: mass None -> 0.09; geometry collision box size=0.1063 0.01 0.01; visual box size=0.1063 0.01 0.01
- link link_rf_3: mass None -> 0.02; geometry collision box size=0.10403 0.01 0.01; visual box size=0.10403 0.01 0.01

Commit message: [feat][ros2][timer]: Add timer

File: Software/Middleware/robot_ros2/src/simulation/urdf/test.urdf (robot description, URDF)
Before this commit: robot 3dof_leg, 14 links, 13 joints
Links:
- removed link world_link
- link body_link: geometry collision box size=0.3 0.14049 0.06; visual box size=0.3 0.18049 0.06
- link link_lb_3: geometry collision sphere radius=0.01; visual box size=0.10403 0.01 0.01
- link link_lf_3: geometry collision sphere radius=0.01; visual box size=0.10403 0.01 0.01
- link link_rb_3: geometry collision sphere radius=0.01; visual box size=0.10403 0.01 0.01
- link link_rf_3: geometry collision sphere radius=0.01; visual box size=0.10403 0.01 0.01
Joints:
- removed joint body_joint
- joint joint_lb_1: limit lower=-1.57 upper= 1.57 effort=   10 velocity=    1 -> lower=-1.57 upper= 1.57 effort= 29.29 velocity= 5
- joint joint_lb_2: limit lower=-6.28 upper=6.28 effort=  10 velocity=   1 -> lower=-6.28 upper= 6.28 effort= 29.29 velocity= 5
- joint joint_lb_3: limit lower=-6.28 upper=6.28 effort=  10 velocity=   1 -> lower=-6.28 upper= 6.28 effort= 19.19 velocity= 10
- joint joint_lf_1: limit lower=-1.57 upper= 1.57 effort=   10 velocity=    1 -> lower=-1.57 upper= 1.57 effort=  29.29 velocity=    5
- joint joint_lf_2: limit lower=-6.28 upper=6.28 effort=  10 velocity=   1 -> lower=-6.28 upper= 6.28 effort=  29.29 velocity=    5
- joint joint_lf_3: limit lower=-6.28 upper=6.28 effort=  10 velocity=   1 -> lower=-6.28 upper= 6.28 effort= 19.19 velocity= 10
- joint joint_rb_1: limit lower=-1.57 upper= 1.57 effort=   10 velocity=    1 -> lower=-1.57 upper= 1.57 effort= 29.29 velocity= 5
- joint joint_rb_2: limit lower=-6.28 upper=6.28 effort=  10 velocity=   1 -> lower=-6.28 upper= 6.28 effort= 29.29 velocity= 5
- joint joint_rb_3: limit lower=-6.28 upper=6.28 effort=  10 velocity=   1 -> lower=-6.28 upper= 6.28 effort= 19.19 velocity= 10
- joint joint_rf_1: limit lower=-1.57 upper= 1.57 effort=   10 velocity=    1 -> lower=-1.57 upper= 1.57 effort= 29.29 velocity= 5
- joint joint_rf_2: limit lower=-6.28 upper=6.28 effort=  10 velocity=   1 -> lower=-6.28 upper=6.28 effort= 29.29 velocity= 5
- joint joint_rf_3: limit lower=-6.28 upper=6.28 effort=  10 velocity=   1 -> lower=-6.28 upper= 6.28 effort= 19.19 velocity= 10

Commit message: [gait]: D-shape

File: Software/Middleware/robot_ros2/src/simulation/urdf/test.urdf (robot description, URDF)
Before this commit: robot 3dof_leg, 13 links, 12 joints
Links:
- link link_lb_1: mass 0.08 -> 0.02
- link link_lb_3: geometry collision box size=0.10403 0.01 0.01; visual box size=0.10403 0.01 0.01
- link link_lf_1: mass 0.08 -> 0.02
- link link_lf_3: geometry collision box size=0.10403 0.01 0.01; visual box size=0.10403 0.01 0.01
- link link_rb_1: mass 0.08 -> 0.02
- link link_rb_3: geometry collision box size=0.10403 0.01 0.01; visual box size=0.10403 0.01 0.01
- link link_rf_1: mass 0.08 -> 0.02
- link link_rf_3: geometry collision box size=0.10403 0.01 0.01; visual box size=0.10403 0.01 0.01

Commit message: [update][ros2][robot-params]: Update the new robot's parameters

File: Software/Middleware/robot_ros2/src/simulation/urdf/test.urdf (robot description, URDF)
Before this commit: robot 3dof_leg, 13 links, 12 joints
Links:
- link body_link: geometry collision box size=0.350 0.222 0.081; visual box size=0.350 0.222 0.081
- link link_lb_1: geometry collision box size=0.01 0.045 0.01; visual box size=0.01 0.045 0.01
- link link_lb_2: geometry collision box size=0.107 0.01 0.01; visual box size=0.107 0.01 0.01
- link link_lb_3: geometry collision box size=0.116 0.01 0.01; visual box size=0.116 0.01 0.01
- link link_lf_1: geometry collision box size=0.01 0.045 0.01; visual box size=0.01 0.045 0.01
- link link_lf_2: geometry collision box size=0.107 0.01 0.01; visual box size=0.107 0.01 0.01
- link link_lf_3: geometry collision box size=0.116 0.01 0.01; visual box size=0.116 0.01 0.01
- link link_rb_1: geometry collision box size=0.01 0.045 0.01; visual box size=0.01 0.045 0.01
- link link_rb_2: geometry collision box size=0.107 0.01 0.01; visual box size=0.107 0.01 0.01
- link link_rb_3: geometry collision box size=0.116 0.01 0.01; visual box size=0.116 0.01 0.01
- link link_rf_1: geometry collision box size=0.01 0.045 0.01; visual box size=0.01 0.045 0.01
- link link_rf_2: geometry collision box size=0.107 0.01 0.01; visual box size=0.107 0.01 0.01
- link link_rf_3: geometry collision box size=0.116 0.01 0.01; visual box size=0.116 0.01 0.01
Joints:
- joint joint_lb_1: origin xyz=-0.11014   0.07169   0.00026 rpy= 0        -1.57     -3.14    -> xyz=-0.125   0.0965   0.00026 rpy= 0        -1.57     -3.14   
- joint joint_lb_2: origin xyz=0    -0.046    0 rpy=1.57  3.14     0 -> xyz=0    -0.045    0 rpy=1.57  3.14     0
- joint joint_lb_3: origin xyz=-0.1063 0 0 rpy= 0      0 0 -> xyz=-0.107 0 0 rpy= 0      0 0
- joint joint_lf_1: origin xyz=0.11014   0.07169   0.00026 rpy=0        -1.57     -3.14    -> xyz=0.125   0.0965   0.00026 rpy=0        -1.57     -3.14   
- joint joint_lf_2: origin xyz=0    -0.046    0 rpy=1.57  3.14     0 -> xyz=0    -0.045    0 rpy=1.57  3.14     0
- joint joint_lf_3: origin xyz=-0.1063 0 0 rpy= 0      0 0 -> xyz=-0.107 0 0 rpy= 0      0 0
- joint joint_rb_1: origin xyz=-0.11014  -0.07169   0.00026 rpy= 0        -1.57      0    -> xyz=-0.125  -0.0965   0.00026 rpy= 0        -1.57      0   
- joint joint_rb_2: origin xyz=0    -0.046   0 rpy=-1.57 0    3.14 -> xyz=0    -0.045   0 rpy=-1.57 0    3.14
- joint joint_rb_3: origin xyz=-0.1063 0 0 rpy= 0      0 0 -> xyz=-0.107 0 0 rpy= 0      0 0
- joint joint_rf_1: origin xyz=0.11014  -0.07169   0.00026 rpy=0        -1.57      0    -> xyz=0.125  -0.0965   0.00026 rpy=0        -1.57      0   
- joint joint_rf_2: origin xyz= 0    -0.046 0    rpy=-1.57  0     3.14 -> xyz= 0    -0.045 0    rpy=-1.57  0     3.14
- joint joint_rf_3: origin xyz=-0.1063 0 0 rpy= 0      0 0 -> xyz=-0.107 0 0 rpy= 0      0 0
