Commit message: [feat][sim][imu]: Keep balance in the zero pose (#55)

File: Software/Middleware/robot_ros2/src/simulation/urdf/quadrupedRobot.urdf (robot description, URDF)
Before this commit: robot 3dof_leg, 13 links, 12 joints
Links:
- added link world_link
Joints:
- added joint body_joint: type fixed, parent world_link, child body_link, origin xyz=0 0 0.2

Commit message: [feat][sim][imu]: Keep balance while trotting (#55)

File: Software/Middleware/robot_ros2/src/simulation/urdf/quadrupedRobot.urdf (robot description, URDF)
Before this commit: robot 3dof_leg, 14 links, 13 joints
Links:
- removed link world_link
Joints:
- removed joint body_joint
