Commit message: [refactor][sim-and-real]: all

File: Software/Middleware/robot_ros2/src/simulation/urdf/quadruped_robot.urdf (robot description, URDF)
Before this commit: robot quadrupedRobot2, 14 links, 13 joints
Links:
- link base_link: geometry collision mesh filename=package://simulation/meshes/base_link.STL; visual mesh filename=package://simulation/meshes/base_link.STL
- link lb_link1: geometry collision mesh filename=package://simulation/meshes/lb_link1.STL; visual mesh filename=package://simulation/meshes/lb_link1.STL
- link lb_link2: geometry collision mesh filename=package://simulation/meshes/lb_link2.STL; visual mesh filename=package://simulation/meshes/lb_link2.STL
- link lb_link3: geometry collision mesh filename=package://simulation/meshes/lb_link3.STL; visual mesh filename=package://simulation/meshes/lb_link3.STL
- link lf_link1: geometry collision mesh filename=package://simulation/meshes/lf_link1.STL; visual mesh filename=package://simulation/meshes/lf_link1.STL
- link lf_link2: geometry collision mesh filename=package://simulation/meshes/lf_link2.STL; visual mesh filename=package://simulation/meshes/lf_link2.STL
- link lf_link3: geometry collision mesh filename=package://simulation/meshes/lf_link3.STL; visual mesh filename=package://simulation/meshes/lf_link3.STL
- link rb_link1: geometry collision mesh filename=package://simulation/meshes/rb_link1.STL; visual mesh filename=package://simulation/meshes/rb_link1.STL
- link rb_link2: geometry collision mesh filename=package://simulation/meshes/rb_link2.STL; visual mesh filename=package://simulation/meshes/rb_link2.STL
- link rb_link3: geometry collision mesh filename=package://simulation/meshes/rb_link3.STL; visual mesh filename=package://simulation/meshes/rb_link3.STL
- link rf_link1: geometry collision mesh filename=package://simulation/meshes/rf_link1.STL; visual mesh filename=package://simulation/meshes/rf_link1.STL
- link rf_link2: geometry collision mesh filename=package://simulation/meshes/rf_link2.STL; visual mesh filename=package://simulation/meshes/rf_link2.STL
- link rf_link3: geometry collision mesh filename=package://simulation/meshes/rf_link3.STL; visual mesh filename=package://simulation/meshes/rf_link3.STL
