Commit message: [feat][sim][imu]: Zero pose -- balance-normal stable-normal (#66)

File: Software/Middleware/robot_ros2/src/simulation/urdf_new/quadrupedRobot2/urdf/quadrupedRobot2.urdf (robot description, URDF)
Before this commit: robot quadrupedRobot2, 14 links, 13 joints
Links:
- link base_link: mass 2.05989698154163 -> 1.0
- link lb_link1: mass 0.231001021795197 -> 0.02
- link lb_link2: mass 0.0747097984739762 -> 0.09
- link lb_link3: mass 0.0172870048509733 -> 0.02
- link lf_link1: mass 0.231001021795197 -> 0.02
- link lf_link2: mass 0.0747097984755013 -> 0.09
- link lf_link3: mass 0.0172870017262757 -> 0.02
- link rb_link1: mass 0.231001021795197 -> 0.02
- link rb_link2: mass 0.0747097984689319 -> 0.09
- link rb_link3: mass 0.0172870064077148 -> 0.02
- link rf_link1: mass 0.231001021795197 -> 0.02
- link rf_link2: mass 0.0747097984676169 -> 0.09
- link rf_link3: mass 0.0172870015239976 -> 0.02
